Commit message: helloworld

File: amr_vehicle_description/urdf/demo01_helloworld.urdf (robot description, URDF)
Before this commit: robot mycar, 1 links, 0 joints
Links:
- added link wheel_1; visual cylinder length=0.05 radius=0.05
- added link wheel_2; visual cylinder length=0.05 radius=0.05
- added link wheel_3; visual cylinder length=0.05 radius=0.05
- added link wheel_4; visual cylinder length=0.05 radius=0.05
- link base_link: geometry visual box size=0.2 .3 .1
Joints:
- added joint base_to_wheel1: type fixed, parent base_link, child wheel_1, origin xyz=0 0 0
- added joint base_to_wheel2: type fixed, parent base_link, child wheel_2, origin xyz=0 0 0
- added joint base_to_wheel3: type fixed, parent base_link, child wheel_3, origin xyz=0 0 0
- added joint base_to_wheel4: type fixed, parent base_link, child wheel_4, origin xyz=0 0 0
